File: PCB/cybr36.kicad_pcb (KiCad board)
At the start: 2 copper layers, 121 x 99.8 mm, 46 parts, among them SW1 SW_Push, SW10 SW_Push, SW11 SW_Push, SW12 SW_Push, SW13 SW_Push, SW14 SW_Push, SW15 SW_Push, SW16 SW_Push, SW17 SW_Push, SW18 SW_Push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

Commit message: power switch added
Parts:
- added SW22: SW_SPST, Button_Switch_SMD:SW_SPDT_PCM12, B.Cu at (200.3, 119.5)
Connections:
- net Net-(SW21-B) renamed RAW
Routing:
- net +BATT: track 103.5 -> 111.1 mm, vias 1 -> 2
- net RAW: track 80.1 -> 84.8 mm, vias 0 -> 1
- net RST: track 63.3 -> 63.9 mm
